File: kicad/v2/PocketTRS.sch (KiCad schematic (older format))
At the start: 40 parts, among them J1 TRS-80, J2 AudioJack3, J3 Mini-DIN-6, J4 DB15_Female_HighDensity, J5 Programmer, J6 USB_B_Micro, J7 PTRS_RESET, J8 ESP_RESET, Q1 BSS138, Q2 MMBT3904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

Commit message: Kicad V2 Fixes for PS/2 Keyboard
Changed PS2_DATA to GPIO32 and PS2_CLK to GPIO33
Connections:
- net PS2_CLK: now also U1.9 (IO33); no longer U1.8 (IO32)
- net PS2_DATA: now also U1.8 (IO32); no longer U1.9 (IO33)
Changed lines of the file:
@@
 	2000 1400 1700 1400
 Text GLabel 1700 1800 0    50   Input ~ 0
+PS2_DATA
+Text GLabel 1150 1900 0    50   Input ~ 0
 PS2_CLK
-Text GLabel 1150 1900 0    50   Input ~ 0
-PS2_DATA
 Text GLabel 1700 2000 0    50   Input ~ 0
 CASS_OUT
